File: FSKmodem2.sch (EAGLE design)
At the start: 9 parts, among them IC1 TCM3105

Commit message: Fixing the resistors, they were so wrong
Parts:
- R1: value 8k06 -> 18k; device rcl:R-EU_0207/7 -> rcl:R-EU_0204/7
- R2: device rcl:R-EU_0207/7 -> rcl:R-EU_0204/7
- R3: value 19k6 -> 33k; device rcl:R-EU_0207/7 -> rcl:R-EU_0204/7
Connections:
- removed net N$10: IC1.RXB, R1.1, R2.2
- removed net N$11: IC1.CDL, R2.1, R3.2
- new net N$1: IC1.CDL, R1.1, R2.2
- new net N$7: IC1.RXB, R2.1, R3.2
Changed lines of the file:
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@@
 <part name="SV2" library="con-lstb" deviceset="MA04-1" device=""/>
 <part name="Q1" library="murata-resonators" deviceset="CSTLS_G" device=""/>
-<part name="R1" library="rcl" deviceset="R-EU_" device="0207/7" value="8k06"/>
-<part name="R2" library="rcl" deviceset="R-EU_" device="0207/7" value="5k6"/>
-<part name="R3" library="rcl" deviceset="R-EU_" device="0207/7" value="19k6"/>
 <part name="C1" library="rcl" deviceset="C-EU" device="050-024X044" value="100n"/>
 <part name="C2" library="rcl" deviceset="C-EU" device="050-024X044" value="100n"/>
+<part name="R1" library="rcl" deviceset="R-EU_" device="0204/7" value="18k"/>
+<part name="R2" library="rcl" deviceset="R-EU_" device="0204/7" value="5k6"/>
+<part name="R3" library="rcl" deviceset="R-EU_" device="0204/7" value="33k"/>
 </parts>
 <sheets>
@@
 <instance part="SV2" gate="1" x="0" y="45.72"/>
 <instance part="Q1" gate="G$1" x="73.66" y="58.42"/>
+<instance part="C1" gate="G$1" x="76.2" y="40.64" rot="R90"/>
+<instance part="C2" gate="G$1" x="68.58" y="35.56" rot="R90"/>
 <instance part="R1" gate="G$1" x="20.32" y="53.34" rot="R90"/>
 <instance part="R2" gate="G$1" x="20.32" y="43.18" rot="R90"/>
 <instance part="R3" gate="G$1" x="20.32" y="33.02" rot="R90"/>
-<instance part="C1" gate="G$1" x="76.2" y="40.64" rot="R90"/>
-<instance part="C2" gate="G$1" x="68.58" y="35.56" rot="R90"/>
 </instances>
 <busses>
@@
 <wire x1="20.32" y1="22.86" x2="7.62" y2="22.86" width="0.1524" layer="91"/>
 <wire x1="7.62" y1="22.86" x2="7.62" y2="40.64" width="0.1524" layer="91"/>
-<wire x1="20.32" y1="27.94" x2="20.32" y2="22.86" width="0.1524" layer="91"/>
-<junction x="20.32" y="22.86"/>
 <junction x="48.26" y="22.86"/>
 <pinref part="SV1" gate="G$1" pin="3"/>
@@
 <junction x="63.5" y="22.86"/>
 <pinref part="R3" gate="G$1" pin="1"/>
+<wire x1="20.32" y1="27.94" x2="20.32" y2="22.86" width="0.1524" layer="91"/>
+<junction x="20.32" y="22.86"/>
 </segment>
 </net>
@@
 <wire x1="7.62" y1="48.26" x2="7.62" y2="71.12" width="0.1524" layer="91"/>
 <wire x1="7.62" y1="71.12" x2="20.32" y2="71.12" width="0.1524" layer="91"/>
+<junction x="48.26" y="71.12"/>
+<pinref part="R1" gate="G$1" pin="2"/>
 <wire x1="20.32" y1="71.12" x2="48.26" y2="71.12" width="0.1524" layer="91"/>
 <wire x1="20.32" y1="58.42" x2="20.32" y2="71.12" width="0.1524" layer="91"/>
 <junction x="20.32" y="71.12"/>
-<junction x="48.26" y="71.12"/>
-<pinref part="R1" gate="G$1" pin="2"/>
 </segment>
 </net>
@@
 </segment>
 </net>
-<net name="N$10" class="0">
-<segment>
-<wire x1="20.32" y1="48.26" x2="25.4" y2="48.26" width="0.1524" layer="91"/>
-<wire x1="25.4" y1="48.26" x2="25.4" y2="43.18" width="0.1524" layer="91"/>
-<pinref part="IC1" gate="G$1" pin="RXB"/>
-<wire x1="25.4" y1="43.18" x2="38.1" y2="43.18" width="0.1524" layer="91"/>
-<pinref part="R1" gate="G$1" pin="1"/>
-<pinref part="R2" gate="G$1" pin="2"/>
-<junction x="20.32" y="48.26"/>
-</segment>
-</net>
-<net name="N$11" class="0">
-<segment>
-<wire x1="20.32" y1="38.1" x2="25.4" y2="38.1" width="0.1524" layer="91"/>
-<wire x1="25.4" y1="38.1" x2="25.4" y2="40.64" width="0.1524" layer="91"/>
-<pinref part="IC1" gate="G$1" pin="CDL"/>
-<wire x1="25.4" y1="40.64" x2="38.1" y2="40.64" width="0.1524" layer="91"/>
-<pinref part="R2" gate="G$1" pin="1"/>
-<pinref part="R3" gate="G$1" pin="2"/>
-<junction x="20.32" y="38.1"/>
-</segment>
-</net>
 <net name="N$2" class="0">
 <segment>
@@
 </segment>
 </net>
+<net name="N$1" class="0">
+<segment>
+<pinref part="R1" gate="G$1" pin="1"/>
+<pinref part="R2" gate="G$1" pin="2"/>
+<wire x1="20.32" y1="48.26" x2="33.02" y2="48.26" width="0.1524" layer="91"/>
+<wire x1="33.02" y1="48.26" x2="33.02" y2="40.64" width="0.1524" layer="91"/>
+<pinref part="IC1" gate="G$1" pin="CDL"/>
+<wire x1="33.02" y1="40.64" x2="38.1" y2="40.64" width="0.1524" layer="91"/>
+<junction x="20.32" y="48.26"/>
+</segment>
+</net>
+<net name="N$7" class="0">
+<segment>
+<pinref part="R2" gate="G$1" pin="1"/>
+<pinref part="R3" gate="G$1" pin="2"/>
+<wire x1="20.32" y1="38.1" x2="27.94" y2="38.1" width="0.1524" layer="91"/>
+<wire x1="27.94" y1="38.1" x2="27.94" y2="43.18" width="0.1524" layer="91"/>
+<pinref part="IC1" gate="G$1" pin="RXB"/>
+<wire x1="27.94" y1="43.18" x2="38.1" y2="43.18" width="0.1524" layer="91"/>
+<junction x="20.32" y="38.1"/>
+</segment>
+</net>

Commit message: Change to 5mm long resistors
This also makes boards smaller ~ 30x17mm
Parts:
- R1, R2, R3: device rcl:R-EU_0204/7 -> rcl:R-EU_0204/5
Changed lines of the file:
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@@
 <?xml version="1.0" encoding="utf-8"?>
 <!DOCTYPE eagle SYSTEM "eagle.dtd">
-<eagle version="6.2">
+<eagle version="7.1.0">
 <drawing>
 <settings>
@@
 <part name="C1" library="rcl" deviceset="C-EU" device="050-024X044" value="100n"/>
 <part name="C2" library="rcl" deviceset="C-EU" device="050-024X044" value="100n"/>
-<part name="R1" library="rcl" deviceset="R-EU_" device="0204/7" value="18k"/>
-<part name="R2" library="rcl" deviceset="R-EU_" device="0204/7" value="5k6"/>
-<part name="R3" library="rcl" deviceset="R-EU_" device="0204/7" value="33k"/>
+<part name="R1" library="rcl" deviceset="R-EU_" device="0204/5" value="18k"/>
+<part name="R2" library="rcl" deviceset="R-EU_" device="0204/5" value="5k6"/>
+<part name="R3" library="rcl" deviceset="R-EU_" device="0204/5" value="33k"/>
 </parts>
 <sheets>
